Commit message: concave added in urdf

File: kuka_coke_description/urdf/table.xacro (robot description, xacro)
@@ -5,5 +5,5 @@
 <robot name="table" xmlns:xacro="http://www.ros.org/wiki/xacro">
   <xacro:macro name="table">
-  <link name="table">
+  <link name="table" concave="yes">
     <inertial>
       <origin
@@ -34,5 +34,5 @@
       </material>
     </visual>
-    <collision>
+    <collision concave="yes">
       <origin
         xyz="0 0 0"
