Commit message: new table urdf added

File: kuka_coke_description/urdf/table_pybullet.urdf (robot description, URDF)
Before this commit: robot table, 1 links, 0 joints
Links:
- added link hole_1, mass 1; collision mesh filename=package://kuka_coke_description/meshes/table_hole.STL; visual mesh filename=package://kuka_coke_description/meshes/table_hole.STL
- added link hole_2, mass 1; collision mesh filename=package://kuka_coke_description/meshes/table_hole.STL; visual mesh filename=package://kuka_coke_description/meshes/table_hole.STL
- added link hole_3, mass 1; collision mesh filename=package://kuka_coke_description/meshes/table_hole.STL; visual mesh filename=package://kuka_coke_description/meshes/table_hole.STL
- added link hole_4, mass 1; collision mesh filename=package://kuka_coke_description/meshes/table_hole.STL; visual mesh filename=package://kuka_coke_description/meshes/table_hole.STL
- link table: geometry collision mesh filename=package://kuka_coke_description/meshes/table_base.STL; visual mesh filename=package://kuka_coke_description/meshes/table_base.STL
Joints:
- added joint joint_1: type fixed, parent table, child hole_1, origin xyz=-0.48 -0.4 1.0 rpy=0 0 0
- added joint joint_2: type fixed, parent table, child hole_2, origin xyz=-0.16 -0.4 1.0 rpy=0 0 0
- added joint joint_3: type fixed, parent table, child hole_3, origin xyz=0.16 -0.4 1.0 rpy=0 0 0
- added joint joint_4: type fixed, parent table, child hole_4, origin xyz=0.48 -0.4 1.0 rpy=0 0 0

Commit message: package and foulder added to params

File: kuka_coke_description/urdf/table_pybullet.urdf (robot description, URDF)
Before this commit: robot table, 5 links, 4 joints
Links:
- removed link hole_1
- removed link hole_2
- removed link hole_3
- removed link hole_4
- link table: geometry collision mesh filename=package://kuka_coke_description/meshes/table.stl; visual mesh filename=package://kuka_coke_description/meshes/table.stl
Joints:
- removed joint joint_1
- removed joint joint_2
- removed joint joint_3
- removed joint joint_4
