Commit message: gazebo removed

File: kuka_coke_description/urdf/kuka_table_rviz.xacro (robot description, xacro)
@@ -3,5 +3,5 @@
   <xacro:include filename="$(find kr_50_r2500_description)/urdf/kr_50_r2500.xacro" />
   <xacro:property name="prefix" value="''" />
-<link name="world"/>
+  <link name="world"/>
   <xacro:kr_50_r2500 prefix="${prefix}"/>
   <joint name="${prefix}world_to_base_link" type="fixed">
@@ -15,9 +15,9 @@
   <xacro:gripper prefix=""/>
   <joint name="${prefix}gripper_joint" type="fixed">
-    <origin xyz="0 0 0.00" rpy="0 0 0"/>
+    <origin xyz="0 0 0.018" rpy="0 0 0"/>
     <parent link="${prefix}flange" />
     <child link="${prefix}gripper_base" />
   </joint>
-  <joint name="fixed" type="fixed">
+  <joint name="table_fixed" type="fixed">
       <origin
         xyz="0 1.5 0"
@@ -28,9 +28,3 @@
   <xacro:include filename="$(find kuka_coke_description)/urdf/table.xacro" />
   <xacro:table/>
-  <gazebo>
-    <plugin name="gazebo_ros_control" filename="libgazebo_ros_control.so">
-      <robotNamespace>/gripper</robotNamespace>
-      <robotSimType>gazebo_ros_control/DefaultRobotHWSim</robotSimType>
-    </plugin>
-  </gazebo>
 </robot>

File: kuka_coke_description/urdf/table.xacro (robot description, xacro)
@@ -3,5 +3,5 @@
      Commit Version: 1.6.0-4-g7f85cfe  Build Version: 1.6.7995.38578
      For more information, please see http://wiki.ros.org/sw_urdf_exporter -->
-<robot xmlns:xacro="http://www.ros.org/wiki/xacro">
+<robot name="table" xmlns:xacro="http://www.ros.org/wiki/xacro">
   <xacro:macro name="table">
   <link name="table">

Commit message: Position between robot and gripper modified

File: kuka_coke_description/urdf/kuka_table_rviz.xacro (robot description, xacro)
@@ -15,5 +15,5 @@
   <xacro:gripper prefix=""/>
   <joint name="${prefix}gripper_joint" type="fixed">
-    <origin xyz="0 0 0.018" rpy="0 0 0"/>
+    <origin xyz="0 0 0.020" rpy="0 0 0"/>
     <parent link="${prefix}flange" />
     <child link="${prefix}gripper_base" />
